Commit message: Adds drivable robot. Some URI and exporting fixes for new models too.

File: swarm_sim/models/agent1/model.urdf (robot description, URDF)
Before this commit: robot agent1, 7 links, 6 joints
Links:
- removed link left_caster
- removed link left_wheel
- removed link right_caster
- removed link right_wheel
- added link lb_wheel, mass .045; collision cylinder length=.0254 radius=.02921; visual cylinder length=.0254 radius=.02921
- added link lf_wheel, mass .045; collision cylinder length=.0254 radius=.02921; visual cylinder length=.0254 radius=.02921
- added link rb_wheel, mass .045; collision cylinder length=.0254 radius=.02921; visual cylinder length=.0254 radius=.02921
- added link rf_wheel, mass .045; collision cylinder length=.0254 radius=.02921; visual cylinder length=.0254 radius=.02921
Joints:
- removed joint left_caster_joint
- removed joint left_wheel_joint
- removed joint right_caster_joint
- removed joint right_wheel_joint
- added joint lb_wheel_joint: type revolute, parent chassis, child lb_wheel, origin xyz=.09779 -.09 -.01079 rpy=0 0 0, axis 0 1 0, limit lower=0 upper=0 effort=0 velocity=0
- added joint lf_wheel_joint: type revolute, parent chassis, child lf_wheel, origin xyz=-.09779 -.09 -.01079 rpy=0 0 0, axis 0 1 0, limit lower=0 upper=0 effort=0 velocity=0
- added joint rb_wheel_joint: type revolute, parent chassis, child rb_wheel, origin xyz=.09779 .09 -.01079 rpy=0 0 0, axis 0 1 0, limit lower=0 upper=0 effort=0 velocity=0
- added joint rf_wheel_joint: type revolute, parent chassis, child rf_wheel, origin xyz=-.09779 .09 -.01079 rpy=0 0 0, axis 0 1 0, limit lower=0 upper=0 effort=0 velocity=0
