Commit message: Update agent model and lidar placement

File: swarm_sim/models/agent1/model.urdf.xacro (robot description, xacro)
@@ -5,24 +5,25 @@
     <!-- base dimensions -->
     <xacro:property name="base_mass" value="2.26796" />
-    <xacro:property name="base_width" value="0.1524" />     <!-- width=y -->
-    <xacro:property name="base_length" value="0.254" />    <!-- length=x -->
+    <xacro:property name="base_width" value="0.381" />     <!-- width=y -->
+    <xacro:property name="base_length" value="0.381" />    <!-- length=x -->
     <xacro:property name="base_height" value="0.04" />     <!-- height=z -->
     <!-- wheel properties -->
-    <xacro:property name="wheel_radius" value="0.02921" />
-    <xacro:property name="wheel_width" value="0.0254" />
+    <xacro:property name="wheel_radius" value="0.05" />
+    <xacro:property name="wheel_width" value="0.045" />
     <!-- differential properties -->
     <xacro:property name="wheel_mass" value="0.45" />
-    <xacro:property name="wheelbase" value="0.19668" />
-    <xacro:property name="track_width" value="0.18" />
+    <xacro:property name="wheelbase" value="0.3048" />
+    <xacro:property name="track_width" value="0.3572" />
     <xacro:property name="wheel_offset_x" value="${wheelbase / 2}" />
-    <xacro:property name="wheel_offset_y" value="${track_width / 2}" />
+    <xacro:property name="wheel_offset_y" value="${(base_width / 2) + (wheel_width / 2)}" />
     <xacro:property name="wheel_offset_z" value="-0.01079" />
     <!-- lidar properties -->
     <xacro:property name="lidar_mass" value="0.830" />
-    <xacro:property name="lidar_height" value="0.0762" />
-    <xacro:property name="lidar_width" value="0.0508" />
+    <xacro:property name="lidar_height" value="0.0408" />
+    <xacro:property name="lidar_length" value="0.096" />
+    <xacro:property name="lidar_width" value="0.0583" />
     <xacro:property name="lidar_offset_x" value="0.0" />
     <xacro:property name="lidar_offset_y" value="0.0" />
-    <xacro:property name="lidar_offset_z" value="0.0481" />
+    <xacro:property name="lidar_offset_z" value="-${(lidar_height/2) + (base_height/2)}" />
     <!-- imu properties -->
     <xacro:property name="imu_offset_x" value="0.0" />
@@ -56,5 +57,5 @@
     <xacro:wheel_joint name="back_right_wheel" x_offset="${wheel_offset_x}" y_offset="${wheel_offset_y}" z_offset="${wheel_offset_z}" reflect_x="-1" reflect_y="-1"/>
     <!-- lidar link -->
-    <xacro:box_total name="laser" mass="${lidar_mass}" width="${lidar_width}" height="${lidar_height}" length="${lidar_width}"/>
+    <xacro:box_total name="laser" mass="${lidar_mass}" width="${lidar_width}" height="${lidar_height}" length="${lidar_length}"/>
     <joint name="laser_joint" type="fixed">
         <gazebo reference="laser_joint">

Commit message: Add grippers, update sim world

File: swarm_sim/models/agent1/model.urdf.xacro (robot description, xacro)
@@ -17,5 +17,5 @@
     <xacro:property name="wheel_offset_x" value="${wheelbase / 2}" />
     <xacro:property name="wheel_offset_y" value="${(base_width / 2) + (wheel_width / 2)}" />
-    <xacro:property name="wheel_offset_z" value="-0.01079" />
+    <xacro:property name="wheel_offset_z" value="-0.03" />
     <!-- lidar properties -->
     <xacro:property name="lidar_mass" value="0.830" />
@@ -25,9 +25,21 @@
     <xacro:property name="lidar_offset_x" value="0.0" />
     <xacro:property name="lidar_offset_y" value="0.0" />
-    <xacro:property name="lidar_offset_z" value="-${(lidar_height/2) + (base_height/2)}" />
+    <xacro:property name="lidar_offset_z" value="${(lidar_height/2) + (base_height/2)}" />
     <!-- imu properties -->
     <xacro:property name="imu_offset_x" value="0.0" />
     <xacro:property name="imu_offset_y" value="0.0" />
     <xacro:property name="imu_offset_z" value="0.0" />
+    <!-- gripper properties -->
+    <xacro:property name="gripper_length" value="0.07"/>
+    <xacro:property name="gripper_width"  value="0.0127"/>
+    <xacro:property name="gripper_height" value="0.0127"/>
+    <!-- gripper a (top and bottom of robot) properties NOTE: These are offset from the JOINT, not base_link -->
+    <xacro:property name="gripper_a_offset_x" value="0"/>
+    <xacro:property name="gripper_a_offset_y" value="${gripper_length/2 + gripper_width} "/>
+    <xacro:property name="gripper_a_offset_z" value="${gripper_height * 2}"/>
+    <!-- gripper b (sides of robot) properties NOTE: These are offset from the JOINT, not base_link -->
+    <xacro:property name="gripper_b_offset_x" value="${gripper_length/2 + gripper_width} "/>
+    <xacro:property name="gripper_b_offset_y" value="0"/>
+    <xacro:property name="gripper_b_offset_z" value="${gripper_height * 2}"/>
     <!--
         Include other xacro files for simulation plugins, Gazebo references, and macros
@@ -56,4 +68,20 @@
     <xacro:wheel name="back_right_wheel" wheel_radius="${wheel_radius}" wheel_width="${wheel_width}" wheel_mass="${wheel_mass}"/>
     <xacro:wheel_joint name="back_right_wheel" x_offset="${wheel_offset_x}" y_offset="${wheel_offset_y}" z_offset="${wheel_offset_z}" reflect_x="-1" reflect_y="-1"/>
+    <xacro:gripper_total name="gripper_1a" mass="0.05" length="${gripper_length}" width="${gripper_width}" height="${gripper_height}" r="0" p="0" y="1.5708" xyz=" ${gripper_a_offset_x} -${gripper_a_offset_y} ${gripper_a_offset_z}"/>
+    <xacro:gripper_positive_joint name="gripper_1a" x_offset="${base_length/2}" y_offset="${base_width/2}" z_offset="0" reflect_x="1" reflect_y="1"/>
+    <xacro:gripper_total name="gripper_1b" mass="0.05" length="${gripper_length}" width="${gripper_width}" height="${gripper_height}" r="0" p="0" y="0" xyz=" -${gripper_b_offset_x} ${gripper_b_offset_y} ${gripper_b_offset_z}"/>
+    <xacro:gripper_negative_joint name="gripper_1b" x_offset="${base_length/2}" y_offset="${base_width/2}" z_offset="0" reflect_x="1" reflect_y="1"/>
+    <xacro:gripper_total name="gripper_2a" mass="0.05" length="${gripper_length}" width="${gripper_width}" height="${gripper_height}" r="0" p="0" y="1.5708" xyz=" -${gripper_a_offset_x} ${gripper_a_offset_y} ${gripper_a_offset_z}"/>
+    <xacro:gripper_negative_joint name="gripper_2a" x_offset="${base_length/2}" y_offset="${base_width/2}" z_offset="0" reflect_x="1" reflect_y="-1"/>
+    <xacro:gripper_total name="gripper_2b" mass="0.05" length="${gripper_length}" width="${gripper_width}" height="${gripper_height}" r="0" p="0" y="0" xyz=" -${gripper_b_offset_x} ${gripper_b_offset_y} ${gripper_b_offset_z}"/>
+    <xacro:gripper_positive_joint name="gripper_2b" x_offset="${base_length/2}" y_offset="${base_width/2}" z_offset="0" reflect_x="1" reflect_y="-1"/>
+    <xacro:gripper_total name="gripper_3a" mass="0.05" length="${gripper_length}" width="${gripper_width}" height="${gripper_height}" r="0" p="0" y="1.5708" xyz=" ${gripper_a_offset_x} -${gripper_a_offset_y} ${gripper_a_offset_z}"/>S
+    <xacro:gripper_negative_joint name="gripper_3a" x_offset="${base_length/2}" y_offset="${base_width/2}" z_offset="0" reflect_x="-1" reflect_y="1"/>
+    <xacro:gripper_total name="gripper_3b" mass="0.05" length="${gripper_length}" width="${gripper_width}" height="${gripper_height}" r="0" p="0" y="0" xyz=" ${gripper_b_offset_x} ${gripper_b_offset_y} ${gripper_b_offset_z}"/>
+    <xacro:gripper_positive_joint name="gripper_3b" x_offset="${base_length/2}" y_offset="${base_width/2}" z_offset="0" reflect_x="-1" reflect_y="1"/>
+    <xacro:gripper_total name="gripper_4a" mass="0.05" length="${gripper_length}" width="${gripper_width}" height="${gripper_height}" r="0" p="0" y="1.5708" xyz=" ${gripper_a_offset_x} ${gripper_a_offset_y} ${gripper_a_offset_z}"/>
+    <xacro:gripper_positive_joint name="gripper_4a" x_offset="${base_length/2}" y_offset="${base_width/2}" z_offset="0" reflect_x="-1" reflect_y="-1"/>
+    <xacro:gripper_total name="gripper_4b" mass="0.05" length="${gripper_length}" width="${gripper_width}" height="${gripper_height}" r="0" p="0" y="0" xyz=" ${gripper_b_offset_x} ${gripper_b_offset_y} ${gripper_b_offset_z}"/>
+    <xacro:gripper_negative_joint name="gripper_4b" x_offset="${base_length/2}" y_offset="${base_width/2}" z_offset="0" reflect_x="-1" reflect_y="-1"/>
     <!-- lidar link -->
     <xacro:box_total name="laser" mass="${lidar_mass}" width="${lidar_width}" height="${lidar_height}" length="${lidar_length}"/>

Commit message: Adds auto-nav feature and refines mapping

File: swarm_sim/models/agent1/model.urdf.xacro (robot description, xacro)
@@ -16,5 +16,5 @@
     <xacro:property name="track_width" value="0.3572" />
     <xacro:property name="wheel_offset_x" value="${wheelbase / 2}" />
-    <xacro:property name="wheel_offset_y" value="${(base_width / 2) + (wheel_width / 2)}" />
+    <xacro:property name="wheel_offset_y" value="${(base_width / 2) - (wheel_width / 2)}" />
     <xacro:property name="wheel_offset_z" value="-0.03" />
     <!-- lidar properties -->

Commit message: tunes stack for real-time auto-nav

File: swarm_sim/models/agent1/model.urdf.xacro (robot description, xacro)
@@ -5,6 +5,6 @@
     <!-- base dimensions -->
     <xacro:property name="base_mass" value="2.26796" />
-    <xacro:property name="base_width" value="0.381" />     <!-- width=y -->
-    <xacro:property name="base_length" value="0.381" />    <!-- length=x -->
+    <xacro:property name="base_width" value="0.483" />     <!-- width=y -->
+    <xacro:property name="base_length" value="0.483" />    <!-- length=x -->
     <xacro:property name="base_height" value="0.04" />     <!-- height=z -->
     <!-- wheel properties -->
