Commit message: Implements mapping and exploration

File: swarm_sim/models/old_agent1/model.urdf (robot description, URDF)
Before this commit: robot agent1, 7 links, 6 joints
Links:
- added link lidar_link; collision box size=0.0508 0.0508 0.0762; visual box size=0.0508 0.0508 0.0762
Joints:
- added joint lidar_joint: type fixed, parent base_link, child lidar_link, origin xyz=0.0 0.0 0.0481 rpy=0 0 0, axis 0 1 0, limit lower=0.0 upper=0.0 effort=0.0 velocity=0.0
